File: v0.4.4d.kicad_pcb (KiCad board)
At the start: 2 copper layers, 152.4 x 127 mm, 25 parts, among them J3 trionic5_header, U1 Olimex_STM32-407_Extension_He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, U2 MCP2515_Breakout, U3 LM1815, U8 LM2940S-5.0/NOPB

Commit message: Changes
Parts:
- added D1: LED, LED_SMD:LED_0603_1608Metric, F.Cu at (-17.8, 134.6)
- added D2: LED, LED_SMD:LED_0603_1608Metric, F.Cu at (-8.80, 134.6)
- added Q1: Q_NMOS_GDS, Package_TO_SOT_SMD:TO-252-2, F.Cu at (-25.9, 137.3)
- added R7: 1k, Resistor_SMD:R_0603_1608Metric, F.Cu at (-17.8, 137.2)
- added R8: 1k, Resistor_SMD:R_0603_1608Metric, F.Cu at (-17.8, 139.7)
- R5: value 10k -> 1k
