File: outputs.kicad_sch (KiCad schematic)
At the start: 0 parts

Commit message: Boards should be placed correctly now
Parts:
- added D1, D10, D11, D12, D13, D16, D17, D18, D3, D4, D5, D6, D7, D8, D9: LED, LED_SMD:LED_0603_1608Metric, symbol Device:LED
- added Q1, Q10, Q11, Q12, Q13, Q14, Q15, Q2, Q3, Q4, Q5, Q6, Q7, Q8, Q9: Q_NMOS_GDS, Package_TO_SOT_SMD:TO-252-2, symbol Device:Q_NMOS_GDS
- added R10, R11, R12, R13, R14, R15, R16, R17, R18, R19, R20, R21, R22, R23, R24, R25, R26, R27, R28, R29, R30, R31, R32, R33, R34, R35, R36, R7, R8, R9: 1k, Resistor_SMD:R_0603_1608Metric, symbol Device:R
Connections:
- new net: D13.1 (K), R30.2
- new net: D10.1 (K), R24.2
- new net: D6.1 (K), R17.2
- new net: D12.1 (K), R29.2
- new net: D3.1 (K), R11.2
- new net: D1.1 (K), R10.2
- new net: D4.1 (K), R12.2
- new net: D7.1 (K), R18.2
- new net: D17.1 (K), R35.2
- new net: D18.1 (K), R36.2
- new net: D16.1 (K), R32.2
- new net: D5.1 (K), R16.2
- new net: D9.1 (K), R23.2
- new net: D11.1 (K), R28.2
- new net: D8.1 (K), R22.2
- new net +3.3V: D1.2 (A), D10.2 (A), D11.2 (A), D12.2 (A), D13.2 (A), D16.2 (A), D17.2 (A), D18.2 (A), D3.2 (A), D4.2 (A), D5.2 (A), D6.2 (A), D7.2 (A), D8.2 (A), D9.2 (A)
- new net GND: Q1.3 (S), Q10.3 (S), Q11.3 (S), Q12.3 (S), Q13.3 (S), Q14.3 (S), Q15.3 (S), Q2.3 (S), Q3.3 (S), Q4.3 (S), Q5.3 (S), Q6.3 (S), Q7.3 (S), Q8.3 (S), Q9.3 (S), R13.2, R14.2, R15.2, R19.2, R20.2, R21.2, R25.2, R26.2, R27.2, R31.2, R33.2, R34.2, R7.2, R8.2, R9.2
- new net MCU_APCB: Q6.1 (G), R15.1
- new net MCU_CHECKENG: Q12.1 (G), R27.1
- new net MCU_FUELRLY: Q15.1 (G), R34.1
- new net MCU_IAC: Q9.1 (G), R21.1
- new net MCU_IGN1: Q2.1 (G), Q3.1 (G), R8.1, R9.1
- new net MCU_IGN2: Q5.1 (G), R14.1
- new net MCU_IGN3: Q8.1 (G), R20.1
- new net MCU_IGN4: Q11.1 (G), R26.1
- new net MCU_INJ1: Q1.1 (G), R7.1
- new net MCU_INJ2: Q4.1 (G), R13.1
- new net MCU_INJ3: Q7.1 (G), R19.1
- new net MCU_INJ4: Q10.1 (G), R25.1
- new net MCU_MAINRLY: Q14.1 (G), R33.1
- new net MCU_SHIFTUP: Q13.1 (G), R31.1
- new net T5_APCA: Q3.2 (D), R12.1
- new net T5_APCB: Q6.2 (D), R18.1
- new net T5_CHECKENG: Q12.2 (D), R30.1
- new net T5_FUELRLY: Q15.2 (D), R36.1
- new net T5_IAC: Q9.2 (D), R24.1
- new net T5_IGN1: Q2.2 (D), R11.1
- new net T5_IGN2: Q5.2 (D), R17.1
- new net T5_IGN3: Q8.2 (D), R23.1
- new net T5_IGN4: Q11.2 (D), R29.1
- new net T5_INJ1: Q1.2 (D), R10.1
- new net T5_INJ2: Q4.2 (D), R16.1
- new net T5_INJ3: Q7.2 (D), R22.1
- new net T5_INJ4: Q10.2 (D), R28.1
- new net T5_MAINRLY: Q14.2 (D), R35.1
- new net T5_SHIFTUP: Q13.2 (D), R32.1

Commit message: Low side drivers mostly in order
Connections:
- net MCU_IGN1: no longer Q3.1 (G), R9.1
- new net MCU_APCA: Q3.1 (G), R9.1
Changed lines of the file:
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@@
     )
   )
-  (global_label "MCU_IGN1" (shape input) (at 43.18 157.48 180) (fields_autoplaced)
+  (global_label "MCU_APCA" (shape input) (at 43.18 157.48 180) (fields_autoplaced)
     (effects (font (size 1.27 1.27)) (justify right))
-    (property "Intersheet References" "${INTERSHEET_REFS}" (id 0) (at 31.4215 157.4006 0)
+    (property "Intersheet References" "${INTERSHEET_REFS}" (id 0) (at 31.1191 157.4006 0)
       (effects (font (size 1.27 1.27)) (justify right) hide)
     )
