File: speeduino_trionic5.kicad_pcb (KiCad board)
At the start: 2 copper layers, 152.4 x 127 mm, 113 parts, among them J3 trionic5_header, Q1 Q_NMOS_GDS, Q10 Q_NMOS_GDS, Q11 Q_NMOS_GDS, Q12 Q_NMOS_GDS, Q13 Q_NMOS_GDS, Q14 Q_NMOS_GDS, Q15 Q_NMOS_GDS, Q2 Q_NMOS_GDS, Q3 Q_NMOS_GDS, Q4 Q_NMOS_GDS, Q5 Q_NMOS_GDS, Q6 Q_NMOS_GDS, Q7 Q_NMOS_GDS, Q8 Q_NMOS_GDS, Q9 Q_NMOS_GDS, U1 Olimex_STM32-407_Extension_He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, U2 MCP2515_Breakout, U3 LM1815, U4 TCAN330, U8 LM2940S-5.0/NOPB

Commit message: Add copper pour and remove fuel ign tab
Routing:
- net CANL: track 84.1 -> 81.9 mm
- net CANH: track 88.3 -> 86.1 mm
- added copper zone on B.Cu, net GND
- added copper zone on F.Cu, net GND
Other:
- outline, holes or cut-outs redrawn
Changed lines of the file:
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@@
     (fp_line (start -1.75 1.4) (end 1.75 1.4) (layer "F.Fab") (width 0.1))
     (fp_line (start -1.75 -0.7) (end -1.75 1.4) (layer "F.Fab") (width 0.1))
-    (pad "1" smd roundrect (at -1.5375 0 180) (size 1.325 2.35) (layers "F.Cu" "F.Paste" "F.Mask") (roundrect_rratio 0.188679)
+    (pad "1" smd roundrect (at -1.5375 0 180) (size 1.325 2.35) (layers "F.Cu" "F.Paste" "F.Mask") (roundrect_rratio 0.1886792453)
       (net 214 "+5V") (pintype "passive"))
-    (pad "2" smd roundrect (at 1.5375 0 180) (size 1.325 2.35) (layers "F.Cu" "F.Paste" "F.Mask") (roundrect_rratio 0.188679)
+    (pad "2" smd roundrect (at 1.5375 0 180) (size 1.325 2.35) (layers "F.Cu" "F.Paste" "F.Mask") (roundrect_rratio 0.1886792453)
       (net 1 "GND") (pintype "passive"))
     (model "${KICAD6_3DMODEL_DIR}/Capacitor_Tantalum_SMD.3dshapes/CP_EIA-3528-21_Kemet-B.wrl"
@@
     (fp_line (start -3.65 2.15) (end 3.65 2.15) (layer "F.Fab") (width 0.1))
     (fp_line (start -2.65 -2.15) (end -3.65 -1.15) (layer "F.Fab") (width 0.1))
-    (pad "1" smd roundrect (at -3.1125 0 90) (size 2.075 2.55) (layers "F.Cu" "F.Paste" "F.Mask") (roundrect_rratio 0.120482)
+    (pad "1" smd roundrect (at -3.1125 0 90) (size 2.075 2.55) (layers "F.Cu" "F.Paste" "F.Mask") (roundrect_rratio 0.1204819277)
       (net 241 "Net-(C17-Pad1)") (pintype "passive"))
-    (pad "2" smd roundrect (at 3.1125 0 90) (size 2.075 2.55) (layers "F.Cu" "F.Paste" "F.Mask") (roundrect_rratio 0.120482)
+    (pad "2" smd roundrect (at 3.1125 0 90) (size 2.075 2.55) (layers "F.Cu" "F.Paste" "F.Mask") (roundrect_rratio 0.1204819277)
       (net 1 "GND") (pintype "passive"))
     (model "${KICAD6_3DMODEL_DIR}/Capacitor_Tantalum_SMD.3dshapes/CP_EIA-7343-31_Kemet-D.wrl"
@@
   (gr_line (start 193.04 27.94) (end 193.04 132.08) (layer "Edge.Cuts") (width 0.05))
   (gr_line (start 175.26 27.94) (end 193.04 27.94) (layer "Edge.Cuts") (width 0.05))
+  (gr_circle (center 179.0192 123.4186) (end 180.1712 123.4186) (layer "Edge.Cuts") (width 0.254) (fill none))
+  (gr_circle (center 46.7106 30.9626) (end 47.8626 30.9626) (layer "Edge.Cuts") (width 0.254) (fill none))
   (gr_line (start 123.952 149.86) (end 40.64 149.86) (layer "Edge.Cuts") (width 0.05))
   (gr_line (start 58.42 27.94) (end 40.64 27.94) (layer "Edge.Cuts") (width 0.05))
@@
   (gr_line (start 193.04 132.08) (end 180.34 132.08) (layer "Edge.Cuts") (width 0.05))
   (gr_line (start 123.952 129.54) (end 123.952 149.86) (layer "Edge.Cuts") (width 0.05))
+  (gr_circle (center 188.7728 32.131) (end 189.9248 32.131) (layer "Edge.Cuts") (width 0.254) (fill none))
   (gr_line (start 175.26 22.86) (end 175.26 27.94) (layer "Edge.Cuts") (width 0.05))
   (gr_line (start 58.42 22.86) (end 58.42 27.94) (layer "Edge.Cuts") (width 0.05))
   (gr_line (start 58.42 22.86) (end 175.26 22.86) (layer "Edge.Cuts") (width 0.05))
+  (gr_circle (center 46.8884 142.0114) (end 48.0404 142.0114) (layer "Edge.Cuts") (width 0.254) (fill none))
   (gr_line (start 40.64 27.94) (end 40.64 149.86) (layer "Edge.Cuts") (width 0.05))
   (gr_text "Arduino_Uno_R3_Shield" (at 68.9315 72.7725) (layer "B.Fab")
@@
   (segment (start 187.381 50.5916) (end 189.6364 48.3362) (width 0.254) (layer "F.Cu") (net 171))
   (segment (start 187.381 54.7425) (end 187.381 50.5916) (width 0.254) (layer "F.Cu") (net 171))
-  (segment (start 128.84 25.98) (end 130.6392 24.1808) (width 0.762) (layer "B.Cu") (net 171))
+  (segment (start 183.2102 32.2834) (end 191.5668 40.64) (width 0.762) (layer "B.Cu") (net 171))
   (segment (start 130.6392 24.1808) (end 169.0624 24.1808) (width 0.762) (layer "B.Cu") (net 171))
+  (segment (start 177.165 32.2834) (end 183.2102 32.2834) (width 0.762) (layer "B.Cu") (net 171))
   (segment (start 191.5668 46.4058) (end 189.6364 48.3362) (width 0.762) (layer "B.Cu") (net 171))
-  (segment (start 177.165 32.2834) (end 186.9186 32.2834) (width 0.762) (layer "B.Cu") (net 171))
-  (segment (start 186.9186 32.2834) (end 191.5668 36.9316) (width 0.762) (layer "B.Cu") (net 171))
-  (segment (start 191.5668 36.9316) (end 191.5668 46.4058) (width 0.762) (layer "B.Cu") (net 171))
   (segment (start 169.0624 24.1808) (end 177.165 32.2834) (width 0.762) (layer "B.Cu") (net 171))
+  (segment (start 128.84 25.98) (end 130.6392 24.1808) (width 0.762) (layer "B.Cu") (net 171))
+  (segment (start 191.5668 40.64) (end 191.5668 46.4058) (width 0.762) (layer "B.Cu") (net 171))
+  (segment (start 134.6392 24.1808) (end 169.0624 24.1808) (width 0.762) (layer "F.Cu") (net 172))
   (segment (start 191.5668 48.9458) (end 189.6364 50.8762) (width 0.762) (layer "F.Cu") (net 172))
+  (segment (start 132.84 25.98) (end 134.6392 24.1808) (width 0.762) (layer "F.Cu") (net 172))
+  (segment (start 183.2102 32.2834) (end 191.5668 40.64) (width 0.762) (layer "F.Cu") (net 172))
+  (segment (start 191.5668 40.64) (end 191.5668 48.9458) (width 0.762) (layer "F.Cu") (net 172))
   (segment (start 188.031 54.7425) (end 188.031 52.4816) (width 0.254) (layer "F.Cu") (net 172))
   (segment (start 169.0624 24.1808) (end 177.165 32.2834) (width 0.762) (layer "F.Cu") (net 172))
-  (segment (start 177.165 32.2834) (end 186.9186 32.2834) (width 0.762) (layer "F.Cu") (net 172))
-  (segment (start 186.9186 32.2834) (end 191.5668 36.9316) (width 0.762) (layer "F.Cu") (net 172))
-  (segment (start 132.84 25.98) (end 134.6392 24.1808) (width 0.762) (layer "F.Cu") (net 172))
   (segment (start 188.031 52.4816) (end 189.6364 50.8762) (width 0.254) (layer "F.Cu") (net 172))
-  (segment (start 134.6392 24.1808) (end 169.0624 24.1808) (width 0.762) (layer "F.Cu") (net 172))
-  (segment (start 191.5668 36.9316) (end 191.5668 48.9458) (width 0.762) (layer "F.Cu") (net 172))
+  (segment (start 177.165 32.2834) (end 183.2102 32.2834) (width 0.762) (layer "F.Cu") (net 172))
   (segment (start 189.6364 50.8762) (end 189.6872 50.8762) (width 0.762) (layer "B.Cu") (net 172))
   (segment (start 145.9938 99.5118) (end 145.9938 100.4212) (width 0.508) (layer "F.Cu") (net 173))
@@
   (segment (start 79.4766 76.4279) (end 79.4254 76.4791) (width 1.27) (layer "F.Cu") (net 241))
   (segment (start 74.6138 72.1827) (end 79.3435 72.1827) (width 1.27) (layer "F.Cu") (net 241))
+  (zone (net 1) (net_name "GND") (layers F&B.Cu) (hatch edge 0.508)
+    (connect_pads (clearance 0.25))
+    (min_thickness 0.254) (filled_areas_thickness no)
+    (fill yes (thermal_gap 0.508) (thermal_bridge_width 0.508))
+    (polygon
+      (pts
+        (xy 230.6574 157.7594)
+        (xy 37.5412 159.9692)
+        (xy 28.702 20.9296)
+        (xy 209.677 6.0198)
+      )
+    )
+  )
 )
