File: speeduino_trionic5.kicad_pcb (KiCad board)
At the start: 2 copper layers, 152.4 x 127 mm, 113 parts, among them J3 trionic5_header, Q1 Q_NMOS_GDS, Q10 Q_NMOS_GDS, Q11 Q_NMOS_GDS, Q12 Q_NMOS_GDS, Q13 Q_NMOS_GDS, Q14 Q_NMOS_GDS, Q15 Q_NMOS_GDS, Q2 Q_NMOS_GDS, Q3 Q_NMOS_GDS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

Commit message: Changes
Parts:
- C2: value 18nF -> 10nF
- R4: value 180k -> 100k
- moved U1 3.81 mm to (106.7, 64.8)
- moved XA2 3.81 mm to (175.3, 128.3)
Routing:
- net GND: track 748.6 -> 708.8 mm
- net MCU_APCA: track 110.3 -> 126.7 mm, vias 3 -> 2
- net MCU_IGN3: track 180.8 -> 167.8 mm, vias 3 -> 4
- net MCU_APCB: track 101.6 -> 112.9 mm, vias 3 -> 2
- net MCU_IGN2: track 172.0 -> 162.1 mm, vias 3 -> 4
- net MCU_IGN1: track 166.9 -> 160.7 mm, vias 3 -> 4
- net MCU_IGN4: track 191.7 -> 186.3 mm
- net +3.3V: track 609.0 -> 613.1 mm
- net +5V: track 362.1 -> 365.7 mm
- net MCU_WBO2: track 203.7 -> 200.2 mm
- net MCU_BAT: track 201.5 -> 204.9 mm
- net MCU_MAP: track 179.9 -> 176.6 mm
- net MCU_MAINRLY: track 153.8 -> 150.6 mm
- net MCU_TPS: track 182.0 -> 179.2 mm
- net MCU_COMB34: track 195.7 -> 198.1 mm
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Other:
- outline, holes or cut-outs redrawn
