File: inputs.kicad_sch (KiCad schematic)
At the start: 12 parts, among them U3 LM1815

Commit message: Changes
Parts:
- removed D1: LED, LED_SMD:LED_0603_1608Metric, symbol Device:LED
- removed R7: 1k, Resistor_SMD:R_0603_1608Metric, symbol Device:R
- added D2: LED, LED_SMD:LED_0603_1608Metric, symbol Device:LED
- R3: JLCPCB (none) -> C217840
- R5: value 10k -> 1k; JLCPCB (none) -> C217840
Connections:
- net GND: now also D2.1 (K)
- net MCU_CPS: now also D2.2 (A)
Changed lines of the file:
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@@
   (junction (at 255.27 40.64) (diameter 0) (color 0 0 0 0)
   )
+  (junction (at 252.73 53.34) (diameter 0) (color 0 0 0 0)
+  )
   (junction (at 204.47 64.77) (diameter 0) (color 0 0 0 0)
   )
@@
   (junction (at 208.28 53.34) (diameter 0) (color 0 0 0 0)
   )
-  (junction (at 252.73 39.37) (diameter 0) (color 0 0 0 0)
-  )
   (junction (at 255.27 30.48) (diameter 0) (color 0 0 0 0)
   )
@@
     (stroke (width 0) (type default) (color 0 0 0 0))
   )
-  (wire (pts (xy 247.65 36.83) (xy 250.19 36.83))
-    (stroke (width 0) (type default) (color 0 0 0 0))
-  )
   (wire (pts (xy 218.44 57.15) (xy 218.44 55.88))
     (stroke (width 0) (type default) (color 0 0 0 0))
   )
-  (wire (pts (xy 247.65 29.21) (xy 247.65 36.83))
-    (stroke (width 0) (type default) (color 0 0 0 0))
-  )
   (wire (pts (xy 227.33 43.18) (xy 213.36 43.18))
     (stroke (width 0) (type default) (color 0 0 0 0))
@@
     (stroke (width 0) (type default) (color 0 0 0 0))
   )
-  (wire (pts (xy 250.19 39.37) (xy 252.73 39.37))
-    (stroke (width 0) (type default) (color 0 0 0 0))
-  )
   (wire (pts (xy 208.28 41.91) (xy 208.28 45.72))
     (stroke (width 0) (type default) (color 0 0 0 0))
   )
-  (wire (pts (xy 229.87 29.21) (xy 227.33 29.21))
-    (stroke (width 0) (type default) (color 0 0 0 0))
-  )
   (wire (pts (xy 208.28 53.34) (xy 208.28 57.15))
     (stroke (width 0) (type default) (color 0 0 0 0))
@@
     (stroke (width 0) (type default) (color 0 0 0 0))
   )
+  (wire (pts (xy 254 46.99) (xy 252.73 45.72))
+    (stroke (width 0) (type default) (color 0 0 0 0))
+  )
   (wire (pts (xy 252.73 45.72) (xy 250.19 45.72))
     (stroke (width 0) (type default) (color 0 0 0 0))
@@
     (stroke (width 0) (type default) (color 0 0 0 0))
   )
-  (wire (pts (xy 227.33 29.21) (xy 227.33 27.94))
-    (stroke (width 0) (type default) (color 0 0 0 0))
-  )
   (polyline (pts (xy 271.78 20.32) (xy 271.78 76.2))
     (stroke (width 0) (type default) (color 0 0 0 0))
   )
-  (wire (pts (xy 237.49 29.21) (xy 240.03 29.21))
-    (stroke (width 0) (type default) (color 0 0 0 0))
-  )
   (wire (pts (xy 267.97 41.91) (xy 267.97 40.64))
     (stroke (width 0) (type default) (color 0 0 0 0))
@@
     (stroke (width 0) (type default) (color 0 0 0 0))
   )
-  (wire (pts (xy 252.73 38.1) (xy 252.73 39.37))
+  (wire (pts (xy 254 54.61) (xy 252.73 53.34))
     (stroke (width 0) (type default) (color 0 0 0 0))
   )
@@
     (stroke (width 0) (type default) (color 0 0 0 0))
   )
-  (wire (pts (xy 250.19 36.83) (xy 250.19 39.37))
-    (stroke (width 0) (type default) (color 0 0 0 0))
-  )
   (wire (pts (xy 199.39 64.77) (xy 204.47 64.77))
     (stroke (width 0) (type default) (color 0 0 0 0))
@@
     (stroke (width 0) (type default) (color 0 0 0 0))
   )
-  (wire (pts (xy 252.73 39.37) (xy 252.73 45.72))
+  (wire (pts (xy 252.73 38.1) (xy 252.73 45.72))
     (stroke (width 0) (type default) (color 0 0 0 0))
   )
@@
       (effects (font (size 1.27 1.27)) (justify left))
     )
-    (property "Value" "10k" (id 1) (at 247.65 35.56 0)
+    (property "Value" "1k" (id 1) (at 247.65 35.56 0)
       (effects (font (size 1.27 1.27)) (justify left))
     )
@@
       (effects (font (size 1.27 1.27)) hide)
     )
-    (pin "1")
-    (pin "2")
-  )
-  (symbol (lib_id "Device:R") (at 243.84 29.21 270) (unit 1)
-    (in_bom yes) (on_board yes)
-    (property "Reference" "R7" (id 0) (at 245.11 25.4 0)
-      (effects (font (size 1.27 1.27)) (justify left))
-    )
-    (property "Value" "1k" (id 1) (at 242.57 24.13 0)
-      (effects (font (size 1.27 1.27)) (justify left))
-    )
-    (property "Footprint" "Resistor_SMD:R_0603_1608Metric" (id 2) (at 243.84 27.432 90)
-      (effects (font (size 1.27 1.27)) hide)
-    )
-    (property "Datasheet" "~" (id 3) (at 243.84 29.21 0)
+    (property "JLCPCB" "C217840" (id 4) (at 252.73 34.29 0)
       (effects (font (size 1.27 1.27)) hide)
     )
@@
       (effects (font (size 1.27 1.27)) hide)
     )
-    (pin "1")
-    (pin "2")
-  )
-  (symbol (lib_id "power:+3.3V") (at 227.33 27.94 0) (unit 1)
-    (in_bom yes) (on_board yes) (fields_autoplaced)
-    (property "Reference" "#PWR0109" (id 0) (at 227.33 31.75 0)
-      (effects (font (size 1.27 1.27)) hide)
-    )
-    (property "Value" "+3.3V" (id 1) (at 227.33 22.86 0))
-    (property "Footprint" "" (id 2) (at 227.33 27.94 0)
-      (effects (font (size 1.27 1.27)) hide)
-    )
-    (property "Datasheet" "" (id 3) (at 227.33 27.94 0)
-      (effects (font (size 1.27 1.27)) hide)
-    )
-    (pin "1")
-  )
-  (symbol (lib_id "Device:LED") (at 233.68 29.21 180) (unit 1)
-    (in_bom yes) (on_board yes) (fields_autoplaced)
-    (property "Reference" "D1" (id 0) (at 235.2675 21.59 0))
-    (property "Value" "LED" (id 1) (at 235.2675 24.13 0))
-    (property "Footprint" "LED_SMD:LED_0603_1608Metric" (id 2) (at 233.68 29.21 0)
-      (effects (font (size 1.27 1.27)) hide)
-    )
-    (property "Datasheet" "~" (id 3) (at 233.68 29.21 0)
+    (property "JLCPCB" "C217840" (id 4) (at 219.71 36.83 0)
       (effects (font (size 1.27 1.27)) hide)
     )
@@
     (pin "1")
   )
+  (symbol (lib_id "Device:LED") (at 254 50.8 90) (unit 1)
+    (in_bom yes) (on_board yes) (fields_autoplaced)
+    (property "Reference" "D2" (id 0) (at 257.81 51.1174 90)
+      (effects (font (size 1.27 1.27)) (justify right))
+    )
+    (property "Value" "LED" (id 1) (at 257.81 53.6574 90)
+      (effects (font (size 1.27 1.27)) (justify right))
+    )
+    (property "Footprint" "LED_SMD:LED_0603_1608Metric" (id 2) (at 254 50.8 0)
+      (effects (font (size 1.27 1.27)) hide)
+    )
+    (property "Datasheet" "~" (id 3) (at 254 50.8 0)
+      (effects (font (size 1.27 1.27)) hide)
+    )
+    (property "JLCPCB" "C126319" (id 4) (at 254 50.8 90)
+      (effects (font (size 1.27 1.27)) hide)
+    )
+    (pin "1")
+    (pin "2")
+  )
   (symbol (lib_id "power:+3.3V") (at 261.62 54.61 0) (unit 1)

Commit message: Boards should be placed correctly now
Parts:
- D2: JLCPCB C126319 -> C84263
Changed lines of the file:
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@@
       (effects (font (size 1.27 1.27)) hide)
     )
-    (property "JLCPCB" "C126319" (id 4) (at 254 50.8 90)
+    (property "JLCPCB" "C84263" (id 4) (at 254 50.8 90)
       (effects (font (size 1.27 1.27)) hide)
     )

Commit message: Add JLCPCB Components
Parts:
- added R37, R41, R42, R43, R44, R48, R49: 10k, Resistor_SMD:R_0603_1608Metric, symbol Device:R
- added R38, R39, R45, R50: 20k, Resistor_SMD:R_0603_1608Metric, symbol Device:R
- added R40, R47: 1k, Resistor_SMD:R_0603_1608Metric, symbol Device:R
- added R46, R51: 40k, Resistor_SMD:R_0603_1608Metric, symbol Device:R
- C1: JLCPCB (none) -> C296015
- C2: value 10nF -> 18nF; JLCPCB (none) -> C424843
- C3: JLCPCB (none) -> C576855
- R1: JLCPCB (none) -> C188125
- R2: JLCPCB (none) -> C2933251
- R4: value 100k -> 180k; JLCPCB (none) -> C100822
- R6: JLCPCB (none) -> C21190
Connections:
- net +3.3V: now also R6.2, R40.2, R43.1, R47.2; no longer R6.1
- net GND: now also R38.1, R44.2, R45.1, R46.1, R50.1, R51.1
- net at C3.1, U3.14 (RCTIMING): now also R6.1; no longer R6.2
- new net MCU_COM34: R49.1, R51.2
- new net MCU_COMB12: R42.1, R46.2
- new net MCU_COOLANT: R47.1
- new net MCU_IAT: R40.1
- new net MCU_KNOCK: R39.2, R43.2, R44.1
- new net MCU_MAP: R37.1, R38.2
- new net MCU_TPS: R41.1, R45.2
- new net MCU_WBO2: R48.1, R50.2
- new net T5_COMB12: R42.2
- new net T5_COMB34: R49.2
- new net T5_KNOCK: R39.1
- new net T5_MAP: R37.2
- new net T5_TPS: R41.2
- new net T5_WBO2: R48.2

Commit message: More changes
Parts:
- added R52, R53: 10k, Resistor_SMD:R_0603_1608Metric, symbol Device:R
- added R54, R55: 40k, Resistor_SMD:R_0603_1608Metric, symbol Device:R
Connections:
- net GND: now also R54.1, R55.1
- new net +15: R52.2
- new net +30: R53.2
- new net MCU_BAT: R53.1, R55.2
- new net MCU_IGN_+15: R52.1, R54.2
Other:
- moved on the sheet: R49, R51

Commit message: Basically done!
Connections:
- net MCU_COM34 renamed MCU_COMB34
Changed lines of the file:
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@@
     )
   )
-  (global_label "MCU_COM34" (shape input) (at 115.57 76.2 0) (fields_autoplaced)
+  (global_label "MCU_COMB34" (shape input) (at 115.57 76.2 0) (fields_autoplaced)
     (effects (font (size 1.27 1.27)) (justify left))
-    (property "Intersheet References" "${INTERSHEET_REFS}" (id 0) (at 129.3847 76.1206 0)
+    (property "Intersheet References" "${INTERSHEET_REFS}" (id 0) (at 130.6547 76.1206 0)
       (effects (font (size 1.27 1.27)) (justify left) hide)
     )

Commit message: More changes
Parts:
- C2: value 18nF -> 10nF
- R4: value 180k -> 100k
Changed lines of the file:
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@@
       (effects (font (size 1.27 1.27)) (justify left))
     )
-    (property "Value" "180k" (id 1) (at 220.98 62.23 0)
+    (property "Value" "100k" (id 1) (at 220.98 62.23 0)
       (effects (font (size 1.27 1.27)) (justify left))
     )
@@
     (in_bom yes) (on_board yes)
     (property "Reference" "C2" (id 0) (at 212.09 59.69 90))
-    (property "Value" "18nF" (id 1) (at 214.63 59.69 90))
+    (property "Value" "10nF" (id 1) (at 214.63 59.69 90))
     (property "Footprint" "Capacitor_SMD:C_0603_1608Metric" (id 2) (at 217.4748 57.15 0)
       (effects (font (size 1.27 1.27)) hide)
