File: speeduino_trionic5.kicad_sch (KiCad schematic)
At the start: 3 parts, among them U1 Olimex_STM32-407_Extension_He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

Commit message: More changes
Connections:
- net +3.3V: now reaches XA1.3V3 (3.3V)
- net +3.3V: now also XA2.3V3 (3.3V)
- net +5V: now reaches XA1.5V1 (5V)
- net +5V: now also XA1.5V3 (5V), XA1.5V4 (5V), XA2.5V1 (5V)
- net MCU_IAT: now reaches XA1.A0
- net MCU_COOLANT: now reaches XA1.A1
- net MCU_TPS: now reaches XA1.A2
- net MCU_MAP: now reaches XA1.A3
- net MCU_BAT: now reaches XA1.A4
- net MCU_WBO2: now reaches XA1.A8
- net MCU_COMB12: now reaches XA1.D18 (D18/TX1)
- net MCU_COMB34: now reaches XA1.D19 (D19/RX1)
- net MCU_IGN_+15: now reaches XA1.D2 (D2_INT0)
- net CAN_INT: now reaches XA1.D20 (D20/SDA)
- net MCU_FUELRLY: now reaches XA1.D22
- net MCU_MAINRLY: now reaches XA1.D23
- net MCU_APCA: now reaches XA1.D44
- net MCU_APCB: now reaches XA1.D45
- net MISO: now reaches XA1.D50 (D50_MISO)
- net MOSI: now reaches XA1.D51 (D51_MOSI)
- net SCK: now reaches XA1.D52 (D52_SCK)
- net CAN_CS: now reaches XA1.D53 (D53_CS)
- net GND: now reaches XA1.GND1 (GND)
- net GND: now also XA1.GND2 (GND), XA1.GND3 (GND), XA1.GND5 (GND), XA1.GND6 (GND), XA2.GND1 (GND), XA2.GND2 (GND), XA2.GND3 (GND)

Commit message: Add stuff
Parts:
- XA1: footprint PCM_arduino-library:Arduino_Mega2560_Shield -> arduino-library:Arduino_Mega2560_Shield
- XA2: footprint PCM_arduino-library:Arduino_Uno_R3_Shield -> arduino-library:Arduino_Uno_R3_Shield
Connections:
- net MCU_BAT: now also XA2.A4
- net MCU_COOLANT: now also XA2.A1
- net MCU_IAT: now also XA2.A0
- net MCU_MAP: now also XA2.A3
- net MCU_TPS: now also XA2.A2
- net MCU_WBO2: now also XA2.A5
- net MCU_CANRX: now reaches XA2.D0 (D0/RX)
- net MCU_CANTX: now reaches XA2.D1 (D1/TX)
Changed lines of the file:
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@@
     (stroke (width 0) (type default) (color 0 0 0 0))
   )
+  (global_label "MCU_MAP" (shape input) (at 129.54 76.2 180) (fields_autoplaced)
+    (effects (font (size 1.27 1.27)) (justify right))
+    (property "Intersheet References" "${INTERSHEET_REFS}" (id 0) (at 118.3863 76.1206 0)
+      (effects (font (size 1.27 1.27)) (justify right) hide)
+    )
+  )
+  (global_label "MCU_BAT" (shape input) (at 129.54 73.66 180) (fields_autoplaced)
+    (effects (font (size 1.27 1.27)) (justify right))
+    (property "Intersheet References" "${INTERSHEET_REFS}" (id 0) (at 118.8701 73.5806 0)
+      (effects (font (size 1.27 1.27)) (justify right) hide)
+    )
+  )
+  (global_label "MCU_CANTX" (shape input) (at 129.54 55.88 180) (fields_autoplaced)
+    (effects (font (size 1.27 1.27)) (justify right))
+    (property "Intersheet References" "${INTERSHEET_REFS}" (id 0) (at 116.3301 55.8006 0)
+      (effects (font (size 1.27 1.27)) (justify right) hide)
+    )
+  )
   (global_label "MCU_INJ3" (shape input) (at 100.33 55.88 0) (fields_autoplaced)
     (effects (font (size 1.27 1.27)) (justify left))
@@
     )
   )
+  (global_label "MCU_TPS" (shape input) (at 129.54 78.74 180) (fields_autoplaced)
+    (effects (font (size 1.27 1.27)) (justify right))
+    (property "Intersheet References" "${INTERSHEET_REFS}" (id 0) (at 118.7491 78.6606 0)
+      (effects (font (size 1.27 1.27)) (justify right) hide)
+    )
+  )
+  (global_label "MCU_CANRX" (shape input) (at 129.54 53.34 180) (fields_autoplaced)
+    (effects (font (size 1.27 1.27)) (justify right))
+    (property "Intersheet References" "${INTERSHEET_REFS}" (id 0) (at 116.0277 53.2606 0)
+      (effects (font (size 1.27 1.27)) (justify right) hide)
+    )
+  )
+  (global_label "MCU_IAT" (shape input) (at 129.54 83.82 180) (fields_autoplaced)
+    (effects (font (size 1.27 1.27)) (justify right))
+    (property "Intersheet References" "${INTERSHEET_REFS}" (id 0) (at 119.5353 83.7406 0)
+      (effects (font (size 1.27 1.27)) (justify right) hide)
+    )
+  )
   (global_label "MCU_INJ4" (shape input) (at 100.33 58.42 0) (fields_autoplaced)
     (effects (font (size 1.27 1.27)) (justify left))
@@
     )
   )
+  (global_label "MCU_WBO2" (shape input) (at 129.54 71.12 180) (fields_autoplaced)
+    (effects (font (size 1.27 1.27)) (justify right))
+    (property "Intersheet References" "${INTERSHEET_REFS}" (id 0) (at 116.9348 71.0406 0)
+      (effects (font (size 1.27 1.27)) (justify right) hide)
+    )
+  )
   (global_label "MCU_MAINRLY" (shape input) (at 100.33 68.58 0) (fields_autoplaced)
     (effects (font (size 1.27 1.27)) (justify left))
@@
     (property "Intersheet References" "${INTERSHEET_REFS}" (id 0) (at 112.0885 43.1006 0)
       (effects (font (size 1.27 1.27)) (justify left) hide)
+    )
+  )
+  (global_label "MCU_COOLANT" (shape input) (at 129.54 81.28 180) (fields_autoplaced)
+    (effects (font (size 1.27 1.27)) (justify right))
+    (property "Intersheet References" "${INTERSHEET_REFS}" (id 0) (at 113.8506 81.2006 0)
+      (effects (font (size 1.27 1.27)) (justify right) hide)
     )
   )
@@
       (effects (font (size 1.524 1.524)))
     )
-    (property "Footprint" "PCM_arduino-library:Arduino_Mega2560_Shield" (id 2) (at 67.31 163.83 0)
+    (property "Footprint" "arduino-library:Arduino_Mega2560_Shield" (id 2) (at 67.31 163.83 0)
       (effects (font (size 1.524 1.524)) hide)
     )
@@
     (pin "3V3")
     (pin "5V1")
-    (pin "5V2")
     (pin "5V3")
     (pin "5V4")
@@
     (pin "GND2")
     (pin "GND3")
-    (pin "GND4")
     (pin "GND5")
     (pin "GND6")
     (pin "IORF")
-    (pin "MISO")
-    (pin "MOSI")
     (pin "RST1")
-    (pin "RST2")
-    (pin "SCK")
     (pin "SCL")
     (pin "SDA")
@@
       (effects (font (size 1.524 1.524)))
     )
-    (property "Footprint" "PCM_arduino-library:Arduino_Uno_R3_Shield" (id 2) (at 154.94 118.11 0)
+    (property "Footprint" "arduino-library:Arduino_Uno_R3_Shield" (id 2) (at 154.94 118.11 0)
       (effects (font (size 1.524 1.524)) hide)
     )
@@
     (pin "3V3")
     (pin "5V1")
-    (pin "5V2")
     (pin "A0")
     (pin "A1")
@@
     (pin "GND2")
     (pin "GND3")
-    (pin "GND4")
     (pin "IORF")
-    (pin "MISO")
-    (pin "MOSI")
     (pin "RST1")
-    (pin "RST2")
-    (pin "SCK")
     (pin "SCL")
     (pin "SDA")
@@
       (reference "#PWR0160") (unit 1) (value "+3.3V") (footprint "")
     )
+    (path "/00000000-0000-0000-0000-00005cdc3535/69f1c3af-aba9-41f3-9359-5cd63804d515"
+      (reference "#PWR0161") (unit 1) (value "GND") (footprint "")
+    )
+    (path "/00000000-0000-0000-0000-00005cdc3535/baa221e7-3e5a-4913-9d1c-062714ac06ad"
+      (reference "#PWR0162") (unit 1) (value "+3.3V") (footprint "")
+    )
     (path "/00000000-0000-0000-0000-00005cd18d89/46ccbee1-4e2a-4bf8-8e1f-6e0ffec1a5d0"
       (reference "C1") (unit 1) (value "1nF") (footprint "Capacitor_SMD:C_0603_1608Metric")
@@
       (reference "U3") (unit 1) (value "LM1815") (footprint "Package_SO:SOIC-14_3.9x8.7mm_P1.27mm")
     )
+    (path "/00000000-0000-0000-0000-00005cdc3535/50a4570c-9d6b-4685-87a8-34989ca07b37"
+      (reference "U4") (unit 1) (value "TCAN330") (footprint "Package_TO_SOT_SMD:SOT-23-8")
+    )
     (path "/00000000-0000-0000-0000-00005cd18ec3/00000000-0000-0000-0000-00005cfc6620"
       (reference "U8") (unit 1) (value "LM2940S-5.0/NOPB") (footprint "Package_TO_SOT_SMD:SOT-223")
     )
     (path "/23c553c0-474e-48ea-9717-5d046a86dbed"
-      (reference "XA1") (unit 1) (value "Arduino_Mega2560_Shield") (footprint "PCM_arduino-library:Arduino_Mega2560_Shield")
+      (reference "XA1") (unit 1) (value "Arduino_Mega2560_Shield") (footprint "arduino-library:Arduino_Mega2560_Shield")
     )
     (path "/3ae2ecba-da25-4af2-bfd2-c505596d3e7f"
-      (reference "XA2") (unit 1) (value "Arduino_Uno_R3_Shield") (footprint "PCM_arduino-library:Arduino_Uno_R3_Shield")
-    )
-  )
+      (reference "XA2") (unit 1) (value "Arduino_Uno_R3_Shield") (footprint "arduino-library:Arduino_Uno_R3_Shield")
+    )
+  )

Commit message: Basically done!
Connections:
- net +3.3V: now also XA1.AREF
- net MCU_APCA: now also XA2.D4
- net MCU_APCB: now also XA2.D5
- net MCU_COMB12: now also XA2.D11
- net MCU_COMB34: now also XA2.D13
- net MCU_CPS: now also XA2.D12
- net MCU_FUELRLY: now also XA2.D7
- net MCU_IGN1: now also U1.32
- net MCU_IGN2: now also U1.34
- net MCU_IGN3: now also U1.36
- net MCU_IGN4: now also U1.37
- net MCU_IGN_+15: now also XA2.D8
- net MCU_INJ1: now also U1.15
- net MCU_INJ2: now also U1.16
- net MCU_INJ3: now also U1.17
- net MCU_INJ4: now also U1.18
- net MCU_MAINRLY: now also XA2.D6
Other:
- note added: "TIM9: APCA APCB TIM3: CPS TIM1: IGN TIM4: INJ"
Changed lines of the file:
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@@
+    (stroke (width 0) (type default) (color 0 0 0 0))
+  )
+  (wire (pts (xy 19.05 109.22) (xy 34.29 109.22))
     (stroke (width 0) (type default) (color 0 0 0 0))
   )
@@
     (stroke (width 0) (type default) (color 0 0 0 0))
   )
+  (wire (pts (xy 19.05 105.41) (xy 19.05 109.22))
+    (stroke (width 0) (type default) (color 0 0 0 0))
+  )
   (wire (pts (xy 21.59 124.46) (xy 21.59 123.19))
     (stroke (width 0) (type default) (color 0 0 0 0))
@@
     (stroke (width 0) (type default) (color 0 0 0 0))
   )
+  (text "TIM9:\nAPCA\nAPCB\nTIM3:\nCPS\nTIM1:\nIGN\nTIM4:\nINJ" (at 181.61 48.26 0)
+    (effects (font (size 1.27 1.27)) (justify left bottom))
+  )
   (global_label "MCU_MAP" (shape input) (at 129.54 76.2 180) (fields_autoplaced)
     (effects (font (size 1.27 1.27)) (justify right))
@@
     )
   )
+  (global_label "MCU_IGN4" (shape input) (at 217.17 86.36 0) (fields_autoplaced)
+    (effects (font (size 1.27 1.27)) (justify left))
+    (property "Intersheet References" "${INTERSHEET_REFS}" (id 0) (at 228.9285 86.2806 0)
+      (effects (font (size 1.27 1.27)) (justify left) hide)
+    )
+  )
+  (global_label "MCU_IGN1" (shape input) (at 207.01 93.98 180) (fields_autoplaced)
+    (effects (font (size 1.27 1.27)) (justify right))
+    (property "Intersheet References" "${INTERSHEET_REFS}" (id 0) (at 195.2515 93.9006 0)
+      (effects (font (size 1.27 1.27)) (justify right) hide)
+    )
+  )
   (global_label "MCU_BAT" (shape input) (at 129.54 73.66 180) (fields_autoplaced)
     (effects (font (size 1.27 1.27)) (justify right))
@@
     )
   )
+  (global_label "MCU_IGN3" (shape input) (at 207.01 88.9 180) (fields_autoplaced)
+    (effects (font (size 1.27 1.27)) (justify right))
+    (property "Intersheet References" "${INTERSHEET_REFS}" (id 0) (at 195.2515 88.8206 0)
+      (effects (font (size 1.27 1.27)) (justify right) hide)
+    )
+  )
   (global_label "MCU_CPS" (shape input) (at 100.33 38.1 0) (fields_autoplaced)
     (effects (font (size 1.27 1.27)) (justify left))
@@
     )
   )
+  (global_label "MCU_INJ2" (shape input) (at 207.01 59.69 180) (fields_autoplaced)
+    (effects (font (size 1.27 1.27)) (justify right))
+    (property "Intersheet References" "${INTERSHEET_REFS}" (id 0) (at 195.5539 59.6106 0)
+      (effects (font (size 1.27 1.27)) (justify right) hide)
+    )
+  )
+  (global_label "MCU_FUELRLY" (shape input) (at 180.34 66.04 0) (fields_autoplaced)
+    (effects (font (size 1.27 1.27)) (justify left))
+    (property "Intersheet References" "${INTERSHEET_REFS}" (id 0) (at 195.6666 65.9606 0)
+      (effects (font (size 1.27 1.27)) (justify left) hide)
+    )
+  )
   (global_label "MCU_FUELRLY" (shape input) (at 100.33 66.04 0) (fields_autoplaced)
     (effects (font (size 1.27 1.27)) (justify left))
@@
     )
   )
+  (global_label "MCU_INJ4" (shape input) (at 207.01 57.15 180) (fields_autoplaced)
+    (effects (font (size 1.27 1.27)) (justify right))
+    (property "Intersheet References" "${INTERSHEET_REFS}" (id 0) (at 195.5539 57.0706 0)
+      (effects (font (size 1.27 1.27)) (justify right) hide)
+    )
+  )
+  (global_label "MCU_COMB34" (shape input) (at 180.34 81.28 0) (fields_autoplaced)
+    (effects (font (size 1.27 1.27)) (justify left))
+    (property "Intersheet References" "${INTERSHEET_REFS}" (id 0) (at 195.4247 81.2006 0)
+      (effects (font (size 1.27 1.27)) (justify left) hide)
+    )
+  )
+  (global_label "MCU_CPS" (shape input) (at 180.34 78.74 0) (fields_autoplaced)
+    (effects (font (size 1.27 1.27)) (justify left))
+    (property "Intersheet References" "${INTERSHEET_REFS}" (id 0) (at 191.4332 78.6606 0)
+      (effects (font (size 1.27 1.27)) (justify left) hide)
+    )
+  )
   (global_label "MCU_IGN4" (shape input) (at 100.33 48.26 0) (fields_autoplaced)
     (effects (font (size 1.27 1.27)) (justify left))
@@
     )
   )
+  (global_label "MCU_MAINRLY" (shape input) (at 180.34 63.5 0) (fields_autoplaced)
+    (effects (font (size 1.27 1.27)) (justify left))
+    (property "Intersheet References" "${INTERSHEET_REFS}" (id 0) (at 195.5456 63.4206 0)
+      (effects (font (size 1.27 1.27)) (justify left) hide)
+    )
+  )
   (global_label "MCU_COMB34" (shape input) (at 34.29 40.64 180) (fields_autoplaced)
     (effects (font (size 1.27 1.27)) (justify right))
@@
     )
   )
+  (global_label "MCU_APCA" (shape input) (at 180.34 58.42 0) (fields_autoplaced)
+    (effects (font (size 1.27 1.27)) (justify left))
+    (property "Intersheet References" "${INTERSHEET_REFS}" (id 0) (at 192.4009 58.3406 0)
+      (effects (font (size 1.27 1.27)) (justify left) hide)
+    )
+  )
   (global_label "MCU_TPS" (shape input) (at 129.54 78.74 180) (fields_autoplaced)
     (effects (font (size 1.27 1.27)) (justify right))
@@
     )
   )
+  (global_label "MCU_INJ3" (shape input) (at 217.17 57.15 0) (fields_autoplaced)
+    (effects (font (size 1.27 1.27)) (justify left))
+    (property "Intersheet References" "${INTERSHEET_REFS}" (id 0) (at 228.6261 57.0706 0)
+      (effects (font (size 1.27 1.27)) (justify left) hide)
+    )
+  )
   (global_label "MCU_IGN_+15" (shape input) (at 100.33 35.56 0) (fields_autoplaced)
     (effects (font (size 1.27 1.27)) (justify left))
@@
     )
   )
+  (global_label "MCU_COMB12" (shape input) (at 180.34 76.2 0) (fields_autoplaced)
+    (effects (font (size 1.27 1.27)) (justify left))
+    (property "Intersheet References" "${INTERSHEET_REFS}" (id 0) (at 195.4247 76.1206 0)
+      (effects (font (size 1.27 1.27)) (justify left) hide)
+    )
+  )
+  (global_label "MCU_INJ1" (shape input) (at 217.17 59.69 0) (fields_autoplaced)
+    (effects (font (size 1.27 1.27)) (justify left))
+    (property "Intersheet References" "${INTERSHEET_REFS}" (id 0) (at 228.6261 59.6106 0)
+      (effects (font (size 1.27 1.27)) (justify left) hide)
+    )
+  )
   (global_label "MCU_BAT" (shape input) (at 34.29 78.74 180) (fields_autoplaced)
     (effects (font (size 1.27 1.27)) (justify right))
@@
     )
   )
+  (global_label "MCU_IGN2" (shape input) (at 207.01 91.44 180) (fields_autoplaced)
+    (effects (font (size 1.27 1.27)) (justify right))
+    (property "Intersheet References" "${INTERSHEET_REFS}" (id 0) (at 195.2515 91.3606 0)
+      (effects (font (size 1.27 1.27)) (justify right) hide)
+    )
+  )
   (global_label "MCU_INJ1" (shape input) (at 100.33 50.8 0) (fields_autoplaced)
     (effects (font (size 1.27 1.27)) (justify left))
@@
     (effects (font (size 1.27 1.27)) (justify left))
     (property "Intersheet References" "${INTERSHEET_REFS}" (id 0) (at 107.2504 137.0806 0)
+      (effects (font (size 1.27 1.27)) (justify left) hide)
+    )
+  )
+  (global_label "MCU_IGN_+15" (shape input) (at 180.34 68.58 0) (fields_autoplaced)
+    (effects (font (size 1.27 1.27)) (justify left))
+    (property "Intersheet References" "${INTERSHEET_REFS}" (id 0) (at 195.848 68.5006 0)
+      (effects (font (size 1.27 1.27)) (justify left) hide)
+    )
+  )
+  (global_label "MCU_APCB" (shape input) (at 180.34 60.96 0) (fields_autoplaced)
+    (effects (font (size 1.27 1.27)) (justify left))
+    (property "Intersheet References" "${INTERSHEET_REFS}" (id 0) (at 192.5823 60.8806 0)
       (effects (font (size 1.27 1.27)) (justify left) hide)
     )
@@
     (pin "9")
   )
+  (symbol (lib_id "power:+3.3V") (at 19.05 105.41 0) (unit 1)
+    (in_bom yes) (on_board yes) (fields_autoplaced)
+    (property "Reference" "#PWR0163" (id 0) (at 19.05 109.22 0)
+      (effects (font (size 1.27 1.27)) hide)
+    )
+    (property "Value" "+3.3V" (id 1) (at 19.05 100.33 0))
+    (property "Footprint" "" (id 2) (at 19.05 105.41 0)
+      (effects (font (size 1.27 1.27)) hide)
+    )
+    (property "Datasheet" "" (id 3) (at 19.05 105.41 0)
+      (effects (font (size 1.27 1.27)) hide)
+    )
+    (pin "1")
+  )
   (symbol (lib_id "power:+5V") (at 123.19 92.71 0) (unit 1)
     (in_bom yes) (on_board yes) (fields_autoplaced)
@@
       (reference "#PWR0162") (unit 1) (value "+3.3V") (footprint "")
     )
+    (path "/b7bda29c-a79b-4a07-9144-60a6903a3a12"
+      (reference "#PWR0163") (unit 1) (value "+3.3V") (footprint "")
+    )
     (path "/00000000-0000-0000-0000-00005cd18d89/46ccbee1-4e2a-4bf8-8e1f-6e0ffec1a5d0"

Commit message: Add copper pour and remove fuel ign tab
Other:
- removed sheet Fuel & Ignition
Changed lines of the file:
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@@
     (pin "1")
   )
-  (sheet (at 19.05 172.72) (size 12.7 13.97) (fields_autoplaced)
+  (sheet (at 22.86 172.72) (size 12.7 13.97) (fields_autoplaced)
     (stroke (width 0) (type solid) (color 0 0 0 0))
     (fill (color 0 0 0 0.0000))
-    (property "Sheet name" "Fuel & Ignition" (id 0) (at 19.05 172.0084 0)
+    (property "Sheet name" "Inputs" (id 0) (at 22.86 172.0084 0)
       (effects (font (size 1.27 1.27)) (justify left bottom))
     )
-    (property "Sheet file" "Fuel_Ignition.kicad_sch" (id 1) (at 19.05 187.2746 0)
+    (property "Sheet file" "inputs.kicad_sch" (id 1) (at 22.86 187.2746 0)
       (effects (font (size 1.27 1.27)) (justify left top))
     )
   )
-  (sheet (at 45.72 172.72) (size 12.7 13.97) (fields_autoplaced)
+  (sheet (at 44.45 172.72) (size 12.7 13.97) (fields_autoplaced)
     (stroke (width 0) (type solid) (color 0 0 0 0))
     (fill (color 0 0 0 0.0000))
-    (property "Sheet name" "Inputs" (id 0) (at 45.72 172.0084 0)
+    (property "Sheet name" "Power" (id 0) (at 44.45 172.0084 0)
       (effects (font (size 1.27 1.27)) (justify left bottom))
     )
-    (property "Sheet file" "inputs.kicad_sch" (id 1) (at 45.72 187.2746 0)
+    (property "Sheet file" "power.kicad_sch" (id 1) (at 44.45 187.2746 0)
       (effects (font (size 1.27 1.27)) (justify left top))
     )
   )
-  (sheet (at 67.31 172.72) (size 12.7 13.97) (fields_autoplaced)
+  (sheet (at 66.04 172.72) (size 12.7 12.7) (fields_autoplaced)
     (stroke (width 0) (type solid) (color 0 0 0 0))
     (fill (color 0 0 0 0.0000))
-    (property "Sheet name" "Power" (id 0) (at 67.31 172.0084 0)
+    (property "Sheet name" "Connector" (id 0) (at 66.04 172.0084 0)
       (effects (font (size 1.27 1.27)) (justify left bottom))
     )
-    (property "Sheet file" "power.kicad_sch" (id 1) (at 67.31 187.2746 0)
+    (property "Sheet file" "connector.kicad_sch" (id 1) (at 66.04 186.0046 0)
       (effects (font (size 1.27 1.27)) (justify left top))
     )
   )
-  (sheet (at 88.9 172.72) (size 12.7 12.7) (fields_autoplaced)
+  (sheet (at 90.17 172.72) (size 12.7 13.97) (fields_autoplaced)
     (stroke (width 0) (type solid) (color 0 0 0 0))
     (fill (color 0 0 0 0.0000))
-    (property "Sheet name" "Connector" (id 0) (at 88.9 172.0084 0)
+    (property "Sheet name" "Outputs" (id 0) (at 90.17 172.0084 0)
       (effects (font (size 1.27 1.27)) (justify left bottom))
     )
-    (property "Sheet file" "connector.kicad_sch" (id 1) (at 88.9 186.0046 0)
+    (property "Sheet file" "outputs.kicad_sch" (id 1) (at 90.17 187.2746 0)
       (effects (font (size 1.27 1.27)) (justify left top))
     )
   )
-  (sheet (at 113.03 172.72) (size 12.7 13.97) (fields_autoplaced)
+  (sheet (at 109.22 172.72) (size 13.97 13.97) (fields_autoplaced)
     (stroke (width 0) (type solid) (color 0 0 0 0))
     (fill (color 0 0 0 0.0000))
-    (property "Sheet name" "Outputs" (id 0) (at 113.03 172.0084 0)
+    (property "Sheet name" "Proto Area" (id 0) (at 109.22 172.0084 0)
       (effects (font (size 1.27 1.27)) (justify left bottom))
     )
-    (property "Sheet file" "outputs.kicad_sch" (id 1) (at 113.03 187.2746 0)
-      (effects (font (size 1.27 1.27)) (justify left top))
-    )
-  )
-  (sheet (at 132.08 172.72) (size 13.97 13.97) (fields_autoplaced)
-    (stroke (width 0) (type solid) (color 0 0 0 0))
-    (fill (color 0 0 0 0.0000))
-    (property "Sheet name" "Proto Area" (id 0) (at 132.08 172.0084 0)
-      (effects (font (size 1.27 1.27)) (justify left bottom))
-    )
-    (property "Sheet file" "proto.kicad_sch" (id 1) (at 132.08 187.2746 0)
+    (property "Sheet file" "proto.kicad_sch" (id 1) (at 109.22 187.2746 0)
       (effects (font (size 1.27 1.27)) (justify left top))
     )
@@
   (sheet_instances
     (path "/" (page "1"))
-    (path "/00000000-0000-0000-0000-00005cd18c17" (page "2"))
     (path "/00000000-0000-0000-0000-00005cd18d89" (page "3"))
     (path "/00000000-0000-0000-0000-00005cd18ec3" (page "4"))
